Commit message: add caster to onshape model.

File: fastbot_description/onshape/robot.urdf (robot description, URDF)
Before this commit: robot fastbot, 7 links, 6 joints
Links:
- removed link base_link
- removed link camera
- removed link motor
- removed link motor_2
- removed link n10_v2
- removed link wheel_left
- removed link wheel_right
- added link fastbot_chassis, mass 0; collision mesh filename=package://fastbot_description/onshape/assets/fastbot_chassi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; visual mesh filename=package://fastbot_description/onshape/assets/fastbot_chassi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
- added link fastbot_motor, mass 0.0339689; collision mesh filename=package://fastbot_description/onshape/assets/fastbot_motor.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; visual mesh filename=package://fastbot_description/onshape/assets/fastbot_motor.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
- added link fastbot_motor_2, mass 0.0339689; collision mesh filename=package://fastbot_description/onshape/assets/fastbot_motor.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; visual mesh filename=package://fastbot_description/onshape/assets/fastbot_motor.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
- added link lslidar_n10, mass 1e-09; collision mesh filename=package://fastbot_description/onshape/assets/lslidar_n10.stl; visual mesh filename=package://fastbot_description/onshape/assets/lslidar_n10.stl
- added link raspicam, mass 1e-09; collision mesh filename=package://fastbot_description/onshape/assets/raspicam.stl; visual mesh filename=package://fastbot_description/onshape/assets/raspicam.stl
- added link wheel_d65x25_v1, mass 1e-09; collision mesh filename=package://fastbot_description/onshape/assets/wheel_d65x25_v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; collision mesh filename=package://fastbot_description/onshape/assets/wheel_d65x25_v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
- added link wheel_d65x25_v1_2, mass 1e-09; collision mesh filename=package://fastbot_description/onshape/assets/wheel_d65x25_v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; collision mesh filename=package://fastbot_description/onshape/assets/wheel_d65x25_v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
Joints:
- joint camera: child camera -> raspicam; origin xyz=0.0105 -0.0668336 0.09765 rpy=-1.5708 1.14468e-45 6.41848e-15 -> xyz=0.00783428 -0.0661426 0.100995 rpy=-1.5708 1.14468e-45 6.41848e-15; parent base_link -> fastbot_chassis
- joint left_motor: child motor_2 -> fastbot_motor_2; origin xyz=0.024 0.0236664 0.02275 rpy=1.5708 -2.96391e-30 -1.5708 -> xyz=0.0213343 0.0243574 0.0260952 rpy=1.5708 -2.96391e-30 -1.5708; parent base_link -> fastbot_chassis
- joint left_wheel: child wheel_left -> wheel_d65x25_v1_2; origin xyz=-0.02 -0.0085 -0.0191 rpy=-1.2326e-32 -1.54074e-33 3.14159 -> xyz=-0.02 -0.0085 -0.0191 rpy=-1.0988e-15 -7.69421e-16 -1.22177; parent motor_2 -> fastbot_motor_2
- joint lidar: child n10_v2 -> lslidar_n10; origin xyz=-0.014 -0.00983363 0.108 rpy=3.14159 1.13983e-46 -3.14159 -> xyz=-0.0166657 -0.00914257 0.111345 rpy=3.14159 1.13983e-46 -3.14159; parent base_link -> fastbot_chassis
- joint right_motor: child motor -> fastbot_motor; origin xyz=-0.024 0.0236664 0.02275 rpy=-1.5708 -2.94692e-47 -1.5708 -> xyz=-0.0266657 0.0243574 0.0260952 rpy=-1.5708 -2.94692e-47 -1.5708; parent base_link -> fastbot_chassis
- joint right_wheel: child wheel_right -> wheel_d65x25_v1; origin xyz=-0.02 0.0085 -0.0191 rpy=4.35106e-30 2.46519e-32 3.14159 -> xyz=-0.02 0.0085 -0.0191 rpy=8.07204e-30 7.24743e-30 -2.18046; parent motor -> fastbot_motor

Commit message: Update robot.urdf with new parts and joints

File: fastbot_description/onshape/robot.urdf (robot description, URDF)
Before this commit: robot fastbot, 7 links, 6 joints
Links:
- added link pololu_ball_caster, mass 1e-09; collision mesh filename=package://fastbot_description/onshape/assets/pololu_ball_ca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; visual mesh filename=package://fastbot_description/onshape/assets/pololu_ball_ca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
Joints:
- added joint caster: type fixed, parent fastbot_chassis, child pololu_ball_caster, origin xyz=-0.0100317 -0.0541426 0.00334516 rpy=0 -0 0, axis 0 0 1, limit effort=10 velocity=10
