Commit message: Barely functional gazebo 11 sim.

File: fastbot_description/models/urdf/fastbot_body.xacro (robot description, xacro)
@@ -1,293 +1,252 @@
 <?xml version="1.0" ?>
+<!-- Generated using onshape-to-robot -->
+<!-- Onshape document_id: 4757b8f98f7afcc7c3655639 -->
 <robot name="fastbot_body" xmlns:xacro="http://ros.org/wiki/xacro">
-  <!-- Define the constant pi -->
   <xacro:property name="PI" value="3.141592653589793" />
   <xacro:macro name="fastbot_body" params="robot_name">
+    <!-- Link fastbot_chassis -->
     <link name="${robot_name}_base_link">
-		<inertial>
-			<origin rpy="0 0 0" xyz="-0.002760040106013823 -0.001188341092731165 0.0718803300182357"/>
-			<mass value="0.5998126574179536"/>
-			<inertia ixx="0.001977" ixy="-1.9e-05" ixz="1.6e-05" iyy="0.001845" iyz="3.1e-05" izz="0.001587"/>
-		</inertial>
-		<visual>
-			<origin rpy="0 0 0" xyz="0 0 0"/>
-			<geometry>
-				<mesh filename="$(find fastbot_description)/models/meshes/base_link.stl" scale="0.001 0.001 0.001"/>
-			</geometry>
-			<material name="grey"/>
-		</visual>
-		<collision>
-			<origin rpy="0 0 0" xyz="0 0 0"/>
-			<geometry>
-				<mesh filename="$(find fastbot_description)/models/meshes/base_link.stl" scale="0.001 0.001 0.001"/>
-			</geometry>
-		</collision>
-	</link>
-	<link name="${robot_name}_wheel_right">
-		<inertial>
-			<origin rpy="0 0 0" xyz="-1.3588436534317516e-07 -0.01588997385974819 2.4327475205837557e-07"/>
-			<mass value="0.23341302374485867"/>
-			<inertia ixx="9.6e-05" ixy="-0.0" ixz="0.0" iyy="0.00016" iyz="0.0" izz="9.6e-05"/>
-		</inertial>
-		<visual>
-			<origin rpy="0 0 0" xyz="-0.0325 0.07073 -0.03245"/>
-			<geometry>
-                <mesh filename="$(find fastbot_description)/models/meshes/wheel_right.stl" scale="0.001 0.001 0.001"/>
-			</geometry>
-			<material name="black"/>
-		</visual>
-		<collision>
-			<origin rpy="0 0 0" xyz="-0.0325 0.07073 -0.03245"/>
-			<geometry>
-                <mesh filename="$(find fastbot_description)/models/meshes/wheel_right.stl" scale="0.001 0.001 0.001"/>
-			</geometry>
-		</collision>
-	</link>
-	<link name="${robot_name}_wheel_left">
-		<inertial>
-			<origin rpy="0 0 0" xyz="-1.3200802984753013e-07 0.015889975585968247 2.563618809944823e-07"/>
-			<mass value="0.2334125809795772"/>
-			<inertia ixx="9.6e-05" ixy="0.0" ixz="0.0" iyy="0.00016" iyz="-0.0" izz="9.6e-05"/>
-		</inertial>
-		<visual>
-			<origin rpy="0 0 0" xyz="-0.0325 -0.07073 -0.03245"/>
-			<geometry>
-                <mesh filename="$(find fastbot_description)/models/meshes/wheel_left.stl" scale="0.001 0.001 0.001"/>
-			</geometry>
-			<material name="black"/>
-		</visual>
-		<collision>
-			<origin rpy="0 0 0" xyz="-0.0325 -0.07073 -0.03245"/>
-			<geometry>
-                <mesh filename="$(find fastbot_description)/models/meshes/wheel_left.stl" scale="0.001 0.001 0.001"/>
-			</geometry>
-		</collision>
-	</link>
-	<link name="${robot_name}_caster">
-		<inertial>
-			<origin rpy="0 0 0" xyz="-0.01100000059604822 -1.4270326137978878e-17 -0.006845279720279717"/>
-			<mass value="0.02931481955170001"/>
-			<inertia ixx="2e-06" ixy="-0.0" ixz="0.0" iyy="2e-06" iyz="-0.0" izz="1e-06"/>
-		</inertial>
-		<visual>
-			<origin rpy="0 0 0" xyz="0.032 -0.0 -0.01915"/>
-			<geometry>
-				<mesh filename="$(find fastbot_description)/models/meshes/caster.stl" scale="0.001 0.001 0.001"/>
-			</geometry>
-			<material name="black"/>
-		</visual>
-		<collision>
-			<origin rpy="0 0 0" xyz="0.032 -0.0 -0.01915"/>
-			<geometry>
-				<mesh filename="$(find fastbot_description)/models/meshes/caster.stl" scale="0.001 0.001 0.001"/>
-			</geometry>
-		</collision>
-	</link>
-	<link name="${robot_name}_lidar_body">
-		<inertial>
-			<origin rpy="0 0 0" xyz="0.04189252309401799 -0.030999999999999896 0.02544713291508699"/>
-			<mass value="0.07136843474102665"/>
-			<inertia ixx="2.3e-05" ixy="0.0" ixz="5e-06" iyy="6.1e-05" iyz="0.0" izz="7.7e-05"/>
-		</inertial>
-		<visual>
-			<origin rpy="0 0 0" xyz="0.022 -0.031 -0.14715"/>
-			<geometry>
-				<mesh filename="$(find fastbot_description)/models/meshes/lidar_body.stl" scale="0.001 0.001 0.001"/>
-			</geometry>
-			<material name="black"/>
-		</visual>
-		<collision>
-			<origin rpy="0 0 0" xyz="0.022 -0.031 -0.14715"/>
-			<geometry>
-				<mesh filename="$(find fastbot_description)/models/meshes/lidar_body.stl" scale="0.001 0.001 0.001"/>
-			</geometry>
-		</collision>
-	</link>
-	<link name="${robot_name}_lidar_motorend">
-		<inertial>
-			<origin rpy="0 0 0" xyz="-1.3877787807814457e-17 7.710435591426653e-18 0.002750000000000058"/>
-			<mass value="0.0005131791599638964"/>
-			<inertia ixx="0.0" ixy="-0.0" ixz="0.0" iyy="0.0" iyz="0.0" izz="0.0"/>
-		</inertial>
-		<visual>
-			<origin rpy="0 0 0" xyz="-0.05 -0.0 -0.18065"/>
-			<geometry>
-                <mesh filename="$(find fastbot_description)/models/meshes/lidar_motorend.stl" scale="0.001 0.001 0.001"/>
-			</geometry>
-			<material name="blue"/>
-		</visual>
-		<collision>
-			<origin rpy="0 0 0" xyz="-0.05 -0.0 -0.18065"/>
-			<geometry>
-                <mesh filename="$(find fastbot_description)/models/meshes/lidar_motorend.stl" scale="0.001 0.001 0.001"/>
-			</geometry>
-		</collision>
-	</link>
-	<link name="${robot_name}_lidar_bottom">
-		<inertial>
-			<origin rpy="0 0 0" xyz="-1.0850529511452296e-17 5.425264755726148e-18 0.007750000000000035"/>
-			<mass value="0.062236577058626265"/>
-			<inertia ixx="1.8e-05" ixy="-0.0" ixz="-0.0" iyy="1.8e-05" iyz="0.0" izz="3.3e-05"/>
-		</inertial>
-		<visual>
-			<origin rpy="0 0 0" xyz="0.0 -0.0 -0.18065"/>
-			<geometry>
-                <mesh filename="$(find fastbot_description)/models/meshes/lidar_bottom.stl" scale="0.001 0.001 0.001"/>
-			</geometry>
-			<material name="blue"/>
-		</visual>
-		<collision>
-			<origin rpy="0 0 0" xyz="0.0 -0.0 -0.18065"/>
-			<geometry>
-				<mesh filename="$(find fastbot_description)/models/meshes/lidar_bottom.stl" scale="0.001 0.001 0.001"/>
-			</geometry>
-		</collision>
-	</link>
-	<link name="${robot_name}_lidar_frame">
-		<inertial>
-			<origin rpy="0 0 0" xyz="-1.2613740557063325e-17 4.204580185687775e-18 0.00500000000000006"/>
-			<mass value="0.040152630360403944"/>
-			<inertia ixx="1.1e-05" ixy="0.0" ixz="0.0" iyy="1.1e-05" iyz="-0.0" izz="2.2e-05"/>
-		</inertial>
-		<visual>
-			<origin rpy="0 0 0" xyz="0.0 -0.0 -0.19615"/>
-			<geometry>
-                <mesh filename="$(find fastbot_description)/models/meshes/lidar_top_${robot_name}.dae" scale="0.001 0.001 0.001"/>
-     		</geometry>
-			<material name="blue"/>
-		</visual>
-		<collision>
-			<origin rpy="0 0 0" xyz="0.0 -0.0 -0.19615"/>
-			<geometry>
-                <mesh filename="$(find fastbot_description)/models/meshes/lidar_top.stl" scale="0.001 0.001 0.001"/>
-			</geometry>
-		</collision>
-	</link>
-	<link name="${robot_name}_gripper">
-		<inertial>
-			<origin rpy="0 0 0" xyz="-1.2613740557063325e-17 4.204580185687775e-18 0.00500000000000006"/>
-			<mass value="0.040152630360403944"/>
-			<inertia ixx="1.1e-05" ixy="0.0" ixz="0.0" iyy="1.1e-05" iyz="-0.0" izz="2.2e-05"/>
-		</inertial>
-		<visual>
-			<origin rpy="0 0 0" xyz="0.0 0.0 0.0"/>
-			<geometry>
-                <mesh filename="$(find fastbot_description)/models/meshes/LG-NS-gripper.dae" scale="1.0 1.0 1.0"/>
-     		</geometry>
-			<material name="black"/>
-		</visual>
-		<collision>
-			<origin rpy="0 0 0" xyz="0.0 0.0 0.0"/>
-			<geometry>
-                <mesh filename="$(find fastbot_description)/models/meshes/LG-NS-gripper.dae" scale="1.0 1.0 1.0"/>
-			</geometry>
-		</collision>
-	</link>
-	<link name="${robot_name}_lidar">
-	</link>
-	<link name="${robot_name}_imu">
-		<inertial>
-			<origin rpy="0 0 0" xyz="-0.005006317892412869 0.010331821776814253 0.0005641458401822869"/>
-			<mass value="0.0005786974233911084"/>
-			<inertia ixx="0.0" ixy="0.0" ixz="-0.0" iyy="0.0" iyz="-0.0" izz="0.0"/>
-		</inertial>
-		<visual>
-			<origin rpy="0 0 0" xyz="-0.04 0.01025 -0.10543"/>
-			<geometry>
-                <mesh filename="$(find fastbot_description)/models/meshes/imu.stl" scale="0.001 0.001 0.001"/>
-			</geometry>
-			<material name="grey"/>
-		</visual>
-		<collision>
-			<origin rpy="0 0 0" xyz="-0.04 0.01025 -0.10543"/>
-			<geometry>
-                <mesh filename="$(find fastbot_description)/models/meshes/imu.stl" scale="0.001 0.001 0.001"/>
-			</geometry>
-		</collision>
-	</link>
-	<link name="${robot_name}_camera">
-		<inertial>
-			<origin rpy="0 0 0" xyz="-0.000736316919000779 9.521361965188852e-15 0.01215919671545948"/>
-			<mass value="0.011070080401829364"/>
-			<inertia ixx="1e-06" ixy="-0.0" ixz="0.0" iyy="1e-06" iyz="0.0" izz="1e-06"/>
-		</inertial>
-		<visual>
-			<origin rpy="0 0 0" xyz="-0.061 -0.0 -0.11515"/>
-			<geometry>
-				<mesh filename="$(find fastbot_description)/models/meshes/camera.stl" scale="0.001 0.001 0.001"/>
-			</geometry>
-			<material name="grey"/>
-		</visual>
-		<collision>
-			<origin rpy="0 0 0" xyz="-0.061 -0.0 -0.11515"/>
-			<geometry>
-				<mesh filename="$(find fastbot_description)/models/meshes/camera.stl" scale="0.001 0.001 0.001"/>
-			</geometry>
-		</collision>
-	</link>
-	<joint name="${robot_name}_motor_right" type="continuous">
-		<origin rpy="0 0 0" xyz="0.0325 -0.07073 0.03245"/>
-		<parent link="${robot_name}_base_link"/>
-		<child link="${robot_name}_wheel_right"/>
-		<axis xyz="0 1 0"/>
-	</joint>
-	<joint name="${robot_name}_motor_left" type="continuous">
-		<origin rpy="0 0 0" xyz="0.0325 0.07073 0.03245"/>
-		<parent link="${robot_name}_base_link"/>
-		<child link="${robot_name}_wheel_left"/>
-		<axis xyz="0 1 0"/>
-	</joint>
-	<joint name="${robot_name}_Rigid3" type="fixed">
-		<origin rpy="0 0 0" xyz="-0.032 0.0 0.01915"/>
-		<parent link="${robot_name}_base_link"/>
-		<child link="${robot_name}_caster"/>
-	</joint>
-	<joint name="${robot_name}_Rigid4" type="fixed">
-		<origin rpy="0 0 3.1416" xyz="-0.022 0.031 0.14715"/>
-		<parent link="${robot_name}_base_link"/>
-		<child link="${robot_name}_lidar_body"/>
-	</joint>
-	<joint name="${robot_name}_Rigid5" type="fixed">
-		<origin rpy="0 0 0" xyz="0.072 -0.031 0.0335"/>
-		<parent link="${robot_name}_lidar_body"/>
-		<child link="${robot_name}_lidar_motorend"/>
-	</joint>
-	<joint name="${robot_name}_Rigid6" type="fixed">
-		<origin rpy="0 0 0" xyz="0.022 -0.031 0.0335"/>
-		<parent link="${robot_name}_lidar_body"/>
-		<child link="${robot_name}_lidar_bottom"/>
-	</joint>
-	<joint name="${robot_name}_Rigid7" type="fixed">
-		<origin rpy="0 0 0" xyz="0.0 0.0 0.0155"/>
-		<parent link="${robot_name}_lidar_bottom"/>
-		<child link="${robot_name}_lidar_frame"/>
-	</joint>
-	<joint name="${robot_name}_lidar_sensor_joint" type="fixed">
-		<origin rpy="0 0 0" xyz="0.0 0.0 0"/>
-		<parent link="${robot_name}_lidar_frame"/>
-		<child link="${robot_name}_lidar"/>
-	</joint>
-	<joint name="${robot_name}_Rigid8" type="fixed">
-		<origin rpy="0 0 0" xyz="0.04 -0.01025 0.10543"/>
-		<parent link="${robot_name}_base_link"/>
-		<child link="${robot_name}_imu"/>
-	</joint>
-	<joint name="${robot_name}_Rigid9" type="fixed">
-		<origin rpy="0 0 0" xyz="0.061 0.0 0.11515"/>
-		<parent link="${robot_name}_base_link"/>
-		<child link="${robot_name}_camera"/>
-	</joint>
-	<joint name="${robot_name}_gripper" type="fixed">
-		<origin rpy="0 0 1.57" xyz="0.1 0.0 0.01"/>
-		<parent link="${robot_name}_base_link"/>
-		<child link="${robot_name}_gripper"/>
-	</joint>
-	<link name="${robot_name}_camera_sensor">
-	</link>
-	<joint name="${robot_name}_Rigid10" type="fixed">
-		<origin rpy="${-PI/2} 0 ${-PI/2}" xyz="0 0 0"/>
-		<parent link="${robot_name}_camera"/>
-		<child link="${robot_name}_camera_sensor"/>
-	</joint>
+        <inertial>
+            <origin xyz="1.61253e-05 0.000669263 0.059916" rpy="0 0 0"/>
+            <mass value="0.24695"/>
+            <inertia ixx="0.000946018" ixy="-8.62213e-08" ixz="-1.4272e-08" iyy="0.000732103" iyz="1.16569e-05" izz="0.000816741"/>
+        </inertial>
+        <!-- Part fastbot_chassis -->
+        <visual>
+            <origin xyz="0.06 -0.0698336 -0.002" rpy="0 -0 3.14159"/>
+            <geometry>
+                <mesh filename="package://fastbot_description/onshape/assets/fastbot_chassis.stl"/>
+            </geometry>
+            <material name="base_link_material">
+                <color rgba="0.262745 0.282353 0.301961 1.0"/>
+            </material>
+        </visual>
+        <collision>
+            <origin xyz="0.06 -0.0698336 -0.002" rpy="0 -0 3.14159"/>
+            <geometry>
+                <mesh filename="package://fastbot_description/onshape/assets/fastbot_chassis.stl"/>
+            </geometry>
+        </collision>
+    </link>
+    <!-- Link motor_1 -->
+    <link name="${robot_name}_motor_1">
+        <inertial>
+            <origin xyz="0.0067446 0.0085 -0.00855065" rpy="0 0 0"/>
+            <mass value="0.0339689"/>
+            <inertia ixx="2.5517e-06" ixy="-3.26147e-15" ixz="-9.70451e-07" iyy="1.80062e-05" iyz="-1.94099e-15" izz="1.80884e-05"/>
+        </inertial>
+        <!-- Part fastbot_motor -->
+        <visual>
+            <origin xyz="0.0935 -0.00775 -0.036" rpy="-1.5708 -1.5708 0"/>
+            <geometry>
+                <mesh filename="package://fastbot_description/onshape/assets/fastbot_motor.stl"/>
+            </geometry>
+            <material name="fastbot_motor_material">
+                <color rgba="0.129412 0.129412 0.129412 1.0"/>
+            </material>
+        </visual>
+        <collision>
+            <origin xyz="0.0935 -0.00775 -0.036" rpy="-1.5708 -1.5708 0"/>
+            <geometry>
+                <mesh filename="package://fastbot_description/onshape/assets/fastbot_motor.stl"/>
+            </geometry>
+        </collision>
+    </link>
+    <!-- Link wheel_right -->
+    <link name="${robot_name}_wheel_right">
+        <inertial>
+            <origin xyz="0 0 0" rpy="0 0 0"/>
+            <mass value="0.03"/>
+            <inertia ixx="0.0001" ixy="0" ixz="0" iyy="0.0001" iyz="0" izz="0.0002"/>
+        </inertial>
+        <!-- Part wheel_right -->
+        <visual>
+            <origin xyz="0.1135 0.0162 0.103475" rpy="1.5708 1.5708 0"/>
+            <geometry>
+                <mesh filename="package://fastbot_description/onshape/assets/wheel_d65x25_v1.stl"/>
+            </geometry>
+            <material name="wheel_right_material">
+                <color rgba="0.290196 0.290196 0.290196 1.0"/>
+            </material>
+        </visual>
+        <collision>
+            <origin xyz="0.1135 0.0162 0.103475" rpy="1.5708 1.5708 0"/>
+            <geometry>
+                <mesh filename="package://fastbot_description/onshape/assets/wheel_d65x25_v1.stl"/>
+            </geometry>
+        </collision>
+        <!-- Part wheel_left -->
+        <visual>
+            <origin xyz="0.1135 0.0162 0.1039" rpy="1.5708 1.5708 0"/>
+            <geometry>
+                <mesh filename="package://fastbot_description/onshape/assets/wheel_d65x25_v1__2.stl"/>
+            </geometry>
+            <material name="wheel_left_material">
+                <color rgba="0.290196 0.290196 0.290196 1.0"/>
+            </material>
+        </visual>
+        <collision>
+            <origin xyz="0.1135 0.0162 0.1039" rpy="1.5708 1.5708 0"/>
+            <geometry>
+                <mesh filename="package://fastbot_description/onshape/assets/wheel_d65x25_v1__2.stl"/>
+            </geometry>
+        </collision>
+    </link>
+    <!-- Joint from motor to wheel_right -->
+    <joint name="${robot_name}_right_wheel" type="continuous">
+        <origin xyz="-0.02 0.0085 -0.0191" rpy="4.35106e-30 2.46519e-32 3.14159"/>
+        <parent link="${robot_name}_motor_1"/>
+        <child link="${robot_name}_wheel_right"/>
+        <axis xyz="0 0 1"/>
+    </joint>
+    <!-- Joint from base_link to motor_1 -->
+    <joint name="${robot_name}_right_motor" type="fixed">
+        <origin xyz="-0.024 0.0236664 0.02275" rpy="-1.5708 -2.94692e-47 -1.5708"/>
+        <parent link="${robot_name}_base_link"/>
+        <child link="${robot_name}_motor_1"/>
+        <axis xyz="0 0 1"/>
+    </joint>
+    <!-- Link motor_2 -->
+    <link name="${robot_name}_motor_2">
+        <inertial>
+            <origin xyz="0.0067446 -0.0085 -0.00855065" rpy="0 0 0"/>
+            <mass value="0.0339689"/>
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