Commit message: latest changes course creation rosject.

File: fastbot_description/models/urdf/fastbot_body.xacro (robot description, xacro)
@@ -2,11 +2,11 @@
 <!-- Generated using onshape-to-robot -->
 <!-- Onshape document_id: 4757b8f98f7afcc7c3655639 -->
-<robot name="fastbot_body" xmlns:xacro="http://ros.org/wiki/xacro">
+<robot name="fastbot" xmlns:xacro="http://ros.org/wiki/xacro">
   <xacro:property name="PI" value="3.141592653589793" />
   <xacro:macro name="fastbot_body" params="robot_name">
-    <!-- Link fastbot_chassis -->
+    <!-- Link base_link -->
     <link name="${robot_name}_base_link">
         <inertial>
-            <origin xyz="1.61253e-05 0.000669263 0.059916" rpy="0 0 0"/>
+            <origin xyz="0 0 0" rpy="0 0 0"/>
             <mass value="0.24695"/>
             <inertia ixx="0.000946018" ixy="-8.62213e-08" ixz="-1.4272e-08" iyy="0.000732103" iyz="1.16569e-05" izz="0.000816741"/>
@@ -14,14 +14,14 @@
         <!-- Part fastbot_chassis -->
         <visual>
-            <origin xyz="0.06 -0.0698336 -0.002" rpy="0 -0 3.14159"/>
+            <origin xyz="0.0573343 -0.0691426 0.00134516" rpy="0 -0 3.14159"/>
             <geometry>
                 <mesh filename="package://fastbot_description/onshape/assets/fastbot_chassis.stl"/>
             </geometry>
-            <material name="base_link_material">
+            <material name="fastbot_chassis_material">
                 <color rgba="0.262745 0.282353 0.301961 1.0"/>
             </material>
         </visual>
         <collision>
-            <origin xyz="0.06 -0.0698336 -0.002" rpy="0 -0 3.14159"/>
+            <origin xyz="0.0573343 -0.0691426 0.00134516" rpy="0 -0 3.14159"/>
             <geometry>
                 <mesh filename="package://fastbot_description/onshape/assets/fastbot_chassis.stl"/>
@@ -29,5 +29,5 @@
         </collision>
     </link>
-    <!-- Link motor_1 -->
+    <!-- Link fastbot_motor -->
     <link name="${robot_name}_motor_1">
         <inertial>
@@ -60,5 +60,5 @@
             <inertia ixx="0.0001" ixy="0" ixz="0" iyy="0.0001" iyz="0" izz="0.0002"/>
         </inertial>
-        <!-- Part wheel_right -->
+        <!-- Part wheel_d65x25_v1 -->
         <visual>
             <origin xyz="0.1135 0.0162 0.103475" rpy="1.5708 1.5708 0"/>
@@ -66,5 +66,5 @@
                 <mesh filename="package://fastbot_description/onshape/assets/wheel_d65x25_v1.stl"/>
             </geometry>
-            <material name="wheel_right_material">
+            <material name="wheel_d65x25_v1_material">
                 <color rgba="0.290196 0.290196 0.290196 1.0"/>
             </material>
@@ -76,36 +76,36 @@
             </geometry>
         </collision>
-        <!-- Part wheel_left -->
-        <visual>
-            <origin xyz="0.1135 0.0162 0.1039" rpy="1.5708 1.5708 0"/>
-            <geometry>
-                <mesh filename="package://fastbot_description/onshape/assets/wheel_d65x25_v1__2.stl"/>
-            </geometry>
-            <material name="wheel_left_material">
-                <color rgba="0.290196 0.290196 0.290196 1.0"/>
-            </material>
-        </visual>
-        <collision>
-            <origin xyz="0.1135 0.0162 0.1039" rpy="1.5708 1.5708 0"/>
-            <geometry>
-                <mesh filename="package://fastbot_description/onshape/assets/wheel_d65x25_v1__2.stl"/>
-            </geometry>
-        </collision>
-    </link>
-    <!-- Joint from motor to wheel_right -->
+        <!-- Part wheel_d65x25_v1_2 -->
+        <visual>
+            <origin xyz="0.1135 0.0162 0.1039" rpy="1.5708 1.5708 0"/>
+            <geometry>
+                <mesh filename="package://fastbot_description/onshape/assets/wheel_d65x25_v1__2.stl"/>
+            </geometry>
+            <material name="wheel_d65x25_v1_2_material">
+                <color rgba="1 0.933333 0.133333 1.0"/>
+            </material>
+        </visual>
+        <collision>
+            <origin xyz="0.1135 0.0162 0.1039" rpy="1.5708 1.5708 0"/>
+            <geometry>
+                <mesh filename="package://fastbot_description/onshape/assets/wheel_d65x25_v1__2.stl"/>
+            </geometry>
+        </collision>
+    </link>
+    <!-- Joint from fastbot_motor to wheel_d65x25_v1 -->
     <joint name="${robot_name}_right_wheel" type="continuous">
-        <origin xyz="-0.02 0.0085 -0.0191" rpy="4.35106e-30 2.46519e-32 3.14159"/>
+        <origin xyz="-0.02 0.0085 -0.0191" rpy="0 0 0"/>
         <parent link="${robot_name}_motor_1"/>
         <child link="${robot_name}_wheel_right"/>
         <axis xyz="0 0 1"/>
     </joint>
-    <!-- Joint from base_link to motor_1 -->
+    <!-- Joint from fastbot_chassis to fastbot_motor -->
     <joint name="${robot_name}_right_motor" type="fixed">
-        <origin xyz="-0.024 0.0236664 0.02275" rpy="-1.5708 -2.94692e-47 -1.5708"/>
+        <origin xyz="-0.0266657 0.0243574 0.0260952" rpy="-1.5708 -2.94692e-47 -1.5708"/>
         <parent link="${robot_name}_base_link"/>
         <child link="${robot_name}_motor_1"/>
         <axis xyz="0 0 1"/>
     </joint>
-    <!-- Link motor_2 -->
+    <!-- Link fastbot_motor_2 -->
     <link name="${robot_name}_motor_2">
         <inertial>
@@ -131,5 +131,5 @@
         </collision>
     </link>
-    <!-- Link wheel_left -->
+    <!-- Link wheel_d65x25_v1_2 -->
     <link name="${robot_name}_wheel_left">
         <inertial>
@@ -145,5 +145,5 @@
             </geometry>
             <material name="wheel_d65x25_v1_3_material">
-                <color rgba="0.290196 0.290196 0.290196 1.0"/>
+                <color rgba="1 0.933333 0.133333 1.0"/>
             </material>
         </visual>
@@ -171,19 +171,19 @@
         </collision>
     </link>
-    <!-- Joint from motor_2 to wheel_left -->
+    <!-- Joint from fastbot_motor_2 to wheel_d65x25_v1_2 -->
     <joint name="${robot_name}_left_wheel" type="continuous">
-        <origin xyz="-0.02 -0.0085 -0.0191" rpy="-1.2326e-32 -1.54074e-33 3.14159"/>
+        <origin xyz="-0.02 -0.0085 -0.0191" rpy="0 0 0"/>
         <parent link="${robot_name}_motor_2"/>
         <child link="${robot_name}_wheel_left"/>
-        <axis xyz="0 0 1"/>
-    </joint>
-    <!-- Joint from base_link to motor_2 -->
+        <axis xyz="0 0 -1"/>
+    </joint>
+    <!-- Joint from fastbot_chassis to fastbot_motor_2 -->
     <joint name="${robot_name}_left_motor" type="fixed">
-        <origin xyz="0.024 0.0236664 0.02275" rpy="1.5708 -2.96391e-30 -1.5708"/>
+        <origin xyz="0.0213343 0.0243574 0.0260952" rpy="1.5708 -2.96391e-30 -1.5708"/>
         <parent link="${robot_name}_base_link"/>
         <child link="${robot_name}_motor_2"/>
         <axis xyz="0 0 1"/>
     </joint>
-    <!-- Link n10_v2 -->
+    <!-- Link lslidar_n10 -->
     <link name="${robot_name}_n10_v2">
         <inertial>
@@ -192,11 +192,11 @@
             <inertia ixx="1e-09" ixy="0" ixz="0" iyy="1e-09" iyz="0" izz="1e-09"/>
         </inertial>
-        <!-- Part n10_v2 -->
+        <!-- Part lslidar_n10 -->
         <visual>
             <origin xyz="-0.074 -0.06 0.11" rpy="-3.14159 5.94511e-32 -8.90522e-65"/>
             <geometry>
-                <mesh filename="package://fastbot_description/onshape/assets/n10_v2.stl"/>
-            </geometry>
-            <material name="n10_v2_material">
+                <mesh filename="package://fastbot_description/onshape/assets/lslidar_n10.stl"/>
+            </geometry>
+            <material name="lslidar_n10_material">
                 <color rgba="0.0980392 0.0980392 0.0980392 1.0"/>
             </material>
@@ -205,17 +205,16 @@
             <origin xyz="-0.074 -0.06 0.11" rpy="-3.14159 5.94511e-32 -8.90522e-65"/>
             <geometry>
-                <mesh filename="package://fastbot_description/onshape/assets/n10_v2.stl"/>
-            </geometry>
-        </collision>
-    </link>
-    <!-- Joint from base_link to n10_v2 -->
+                <mesh filename="package://fastbot_description/onshape/assets/lslidar_n10.stl"/>
+            </geometry>
+        </collision>
+    </link>
+    <!-- Joint from fastbot_chassis to lslidar_n10 -->
     <joint name="${robot_name}_lidar" type="fixed">
-        <origin xyz="-0.014 -0.00983363 0.108" rpy="3.14159 1.13983e-46 -3.14159"/>
+        <origin xyz="-0.0166657 -0.00914257 0.111345" rpy="3.14159 1.13983e-46 -3.14159"/>
         <parent link="${robot_name}_base_link"/>
         <child link="${robot_name}_n10_v2"/>
         <axis xyz="0 0 1"/>
-        <limit effort="10" velocity="10"/>
-    </joint>
-    <!-- Link camera -->
+    </joint>
+    <!-- Link raspicam -->
     <link name="${robot_name}_camera">
         <inertial>
@@ -224,11 +223,11 @@
             <inertia ixx="1e-09" ixy="0" ixz="0" iyy="1e-09" iyz="0" izz="1e-09"/>
         </inertial>
-        <!-- Part camera -->
+        <!-- Part raspicam -->
         <visual>
             <origin xyz="-0.0105 0.0125 -0.00212" rpy="3.14159 -3.05067e-31 -1.55575e-61"/>
             <geometry>
-                <mesh filename="package://fastbot_description/onshape/assets/part_33.stl"/>
-            </geometry>
-            <material name="camera_material">
+                <mesh filename="package://fastbot_description/onshape/assets/raspicam.stl"/>
+            </geometry>
+            <material name="raspicam_material">
                 <color rgba="0.34902 0.376471 0.4 1.0"/>
             </material>
@@ -237,15 +236,45 @@
             <origin xyz="-0.0105 0.0125 -0.00212" rpy="3.14159 -3.05067e-31 -1.55575e-61"/>
             <geometry>
-                <mesh filename="package://fastbot_description/onshape/assets/part_33.stl"/>
-            </geometry>
-        </collision>
-    </link>
-    <!-- Joint from base_link to camera -->
+                <mesh filename="package://fastbot_description/onshape/assets/raspicam.stl"/>
+            </geometry>
+        </collision>
+    </link>
+    <!-- Joint from fastbot_chassis to raspicam -->
     <joint name="${robot_name}_camera" type="fixed">
-        <origin xyz="0.0105 -0.0668336 0.09765" rpy="-1.5708 1.14468e-45 6.41848e-15"/>
+        <origin xyz="0.00783428 -0.0661426 0.100995" rpy="-1.5708 1.14468e-45 6.41848e-15"/>
         <parent link="${robot_name}_base_link"/>
         <child link="${robot_name}_camera"/>
         <axis xyz="0 0 1"/>
-        <limit effort="10" velocity="10"/>
+    </joint>
+    <!-- Link pololu_ball_caster -->
+    <link name="${robot_name}_ball_caster">
+        <inertial>
+            <origin xyz="0 0 0" rpy="0 0 0"/>
+            <mass value="0.01"/>
+            <inertia ixx="1e-09" ixy="0" ixz="0" iyy="1e-09" iyz="0" izz="1e-09"/>
+        </inertial>
+        <!-- Part pololu_ball_caster -->
+        <visual>
+            <origin xyz="0.006731 0 -0.0106945" rpy="-1.5708 -0 0"/>
+            <geometry>
+                <mesh filename="package://fastbot_description/onshape/assets/pololu_ball_caster.stl"/>
+            </geometry>
+            <material name="pololu_ball_caster_material">
+                <color rgba="0.34902 0.376471 0.4 1.0"/>
+            </material>
+        </visual>
+        <collision>
+            <origin xyz="0.006731 0 -0.0106945" rpy="-1.5708 -0 0"/>
+            <geometry>
+                <mesh filename="package://fastbot_description/onshape/assets/pololu_ball_caster.stl"/>
+            </geometry>
+        </collision>
+    </link>
+    <!-- Joint from fastbot_chassis to pololu_ball_caster -->
+    <joint name="caster" type="fixed">
+        <origin xyz="-0.0100317 -0.0541426 0.00334516" rpy="0 -0 0"/>
+        <parent link="${robot_name}_base_link"/>
+        <child link="${robot_name}_ball_caster"/>
+        <axis xyz="0 0 1"/>
     </joint>
   </xacro:macro>

Commit message: Fixed lidar plugin and added rviz config.

File: fastbot_description/models/urdf/fastbot_body.xacro (robot description, xacro)
@@ -186,9 +186,9 @@
     </joint>
     <!-- Link lslidar_n10 -->
-    <link name="${robot_name}_n10_v2">
+    <link name="${robot_name}_lidar">
         <inertial>
             <origin xyz="0 0 0" rpy="0 0 0"/>
             <mass value="0.05"/>
-            <inertia ixx="1e-09" ixy="0" ixz="0" iyy="1e-09" iyz="0" izz="1e-09"/>
+            <inertia ixx="0.0001" ixy="0" ixz="0" iyy="0.0001" iyz="0" izz="0.0002"/>
         </inertial>
         <!-- Part lslidar_n10 -->
@@ -213,5 +213,5 @@
         <origin xyz="-0.0166657 -0.00914257 0.111345" rpy="3.14159 1.13983e-46 -3.14159"/>
         <parent link="${robot_name}_base_link"/>
-        <child link="${robot_name}_n10_v2"/>
+        <child link="${robot_name}_lidar"/>
         <axis xyz="0 0 1"/>
     </joint>

Commit message: added changes from course creation rosject.

File: fastbot_description/models/urdf/fastbot_body.xacro (robot description, xacro)
@@ -211,5 +211,5 @@
     <!-- Joint from fastbot_chassis to lslidar_n10 -->
     <joint name="${robot_name}_lidar" type="fixed">
-        <origin xyz="-0.0166657 -0.00914257 0.111345" rpy="3.14159 1.13983e-46 -3.14159"/>
+        <origin xyz="-0.0166657 0 0.112" rpy="3.14159 1.13983e-46 -3.14159"/>
         <parent link="${robot_name}_base_link"/>
         <child link="${robot_name}_lidar"/>
@@ -242,5 +242,5 @@
     <!-- Joint from fastbot_chassis to raspicam -->
     <joint name="${robot_name}_camera" type="fixed">
-        <origin xyz="0.00783428 -0.0661426 0.100995" rpy="-1.5708 1.14468e-45 6.41848e-15"/>
+        <origin xyz="0.00783428 -0.0661426 0.100995" rpy="0 0 -1.5708"/>
         <parent link="${robot_name}_base_link"/>
         <child link="${robot_name}_camera"/>

Commit message: Fixed strange movement and physics issues

File: fastbot_description/models/urdf/fastbot_body.xacro (robot description, xacro)
@@ -10,5 +10,5 @@
             <origin xyz="0 0 0" rpy="0 0 0"/>
             <mass value="0.24695"/>
-            <inertia ixx="0.000946018" ixy="-8.62213e-08" ixz="-1.4272e-08" iyy="0.000732103" iyz="1.16569e-05" izz="0.000816741"/>
+            <inertia ixx="0.0007665739583333334" ixy="0.0" ixz="0.0" iyy="0.0005684994791666666" iyz="0.0" izz="0.0007907544791666667"/>
         </inertial>
         <!-- Part fastbot_chassis -->
@@ -24,6 +24,8 @@
         <collision>
             <origin xyz="0.0573343 -0.0691426 0.00134516" rpy="0 -0 3.14159"/>
+            <!--<origin xyz="0.0 0.0 -0.00134516" rpy="0 0 0"/>-->
             <geometry>
                 <mesh filename="package://fastbot_description/onshape/assets/fastbot_chassis.stl"/>
+                <!--<box size="0.12 0.155 0.115" />-->
             </geometry>
         </collision>
@@ -58,5 +60,5 @@
             <origin xyz="0 0 0" rpy="0 0 0"/>
             <mass value="0.03"/>
-            <inertia ixx="0.0001" ixy="0" ixz="0" iyy="0.0001" iyz="0" izz="0.0002"/>
+            <inertia ixx="1.0444293461874998e-05" ixy="0" ixz="0" iyy="1.0444293461874998e-05" iyz="0" izz="1.7812890903749995e-05"/>
         </inertial>
         <!-- Part wheel_d65x25_v1 -->
@@ -136,5 +138,5 @@
             <origin xyz="0 0 0" rpy="0 0 0"/>
             <mass value="0.03"/>
-            <inertia ixx="0.0001" ixy="0" ixz="0" iyy="0.0001" iyz="0" izz="0.0002"/>
+            <inertia ixx="1.0444293461874998e-05" ixy="0" ixz="0" iyy="1.0444293461874998e-05" iyz="0" izz="1.7812890903749995e-05"/>
         </inertial>
         <!-- Part wheel_d65x25_v1_3 -->
@@ -254,5 +256,4 @@
             <inertia ixx="1e-09" ixy="0" ixz="0" iyy="1e-09" iyz="0" izz="1e-09"/>
         </inertial>
-        <!-- Part pololu_ball_caster -->
         <visual>
             <origin xyz="0.006731 0 -0.0106945" rpy="-1.5708 -0 0"/>
